File: hardware_v2/pcb/kapula.kicad_sch (KiCad schematic)
At the start: 166 parts, among them J1 Conn_02x10_Odd_Even, J2 Conn_02x10_Odd_Even, J3 U.FL, J4 U.FL, J5 U.FL, J6 U.FL, Q1 AO3401A, Q1 BSS84, Q2 AO3400A, Q3 AO3400A, Q4 AO3400A, Q5 AO3401A, T1 BW21S7511A01TF, T2 BW21S7511A01TF, T3 BW21S7511A01TF, T4 BW21S7511A01TF, U1 TP4054, U2 DW01+G, U3 XC6206P332MR, U4 FM8002A, U5 EFR32FG14P233F256GM48-B, U6 TG2016SMN 38.4000M-MCGNNM3, U7 XA213-G4J, Y1 32768 Hz

Commit message: 0
Parts:
- renumbered Q1 to Q6
